Commit message: add octomap_server and it works good

File: src/husky_description/urdf/accessories/vlp.urdf.xacro (robot description, xacro)
@@ -21,8 +21,8 @@
 ARISING IN ANY WAY OUT OF THE USE OF THIS SOFTWARE, EVEN IF ADVISED OF THE POSSIBILITY OF SUCH DAMAGE.
 -->
+<!-- Linxius
 <robot name="husky_robot" xmlns:xacro="http://ros.org/wiki/xacro">
-  <xacro:arg name="laser_enabled" default="$(optenv HUSKY_LMS1XX_ENABLED false)" />
-  <xacro:arg name="ur5_enabled" default="$(optenv HUSKY_UR5_ENABLED false)" />
-  <xacro:arg name="kinect_enabled" default="false" />
+-->
+<robot xmlns:xacro="http://ros.org/wiki/xacro">
   <xacro:arg name="hesai_lidar_enabled" default="true" />
   <!-- Linxius
@@ -86,4 +86,6 @@
   </xacro:macro>
   <xacro:velodyne_lidar />
+  <!-- Linxius
   <xacro:husky_robot />
+  -->
 </robot>

File: src/husky_description/urdf/husky.urdf.xacro (robot description, xacro)
@@ -39,4 +39,6 @@
   <xacro:include filename="$(find husky_description)/urdf/accessories/sick_lms1xx_mount.urdf.xacro"/>
   <xacro:include filename="$(find husky_description)/urdf/accessories/sensor_arch.urdf.xacro"/>
+  <!-- Linxius -->
+  <xacro:include filename="$(find husky_description)/urdf/accessories/vlp.urdf.xacro"/>
   <xacro:property name="M_PI" value="3.14159"/>
   <!-- Base Size -->
@@ -136,59 +138,4 @@
     <xacro:kinect_camera prefix="camera" robot_namespace="$(arg robot_namespace)"/>
   </xacro:if>
-  <!-- Linxius -->
-  <xacro:macro name="velodyne_lidar">
-    <xacro:property name="M_PI" value="3.1415926535897931" />
-    <!--<xacro:include filename="$(find velodyne_description)/urdf/HDL-32E.urdf.xacro"/>
-        <HDL-32E parent="base_link"
-        name="velodyne2"
-        topic="/velodyne_points2"
-        hz="10"
-        samples ="2000"
-        lasers="40">
-        <origin xyz="0 0 0.6" rpy="0 0 0"/>
-        </HDL-32E>-->
-    <xacro:include filename="$(find velodyne_description)/urdf/VLP-16.urdf.xacro"/>
-    <!--
-        samples="440"
-        lasers="16"
-        max_range ="130.0"
-        noise ="0.008"
-    -->
-    <!--For Hesai 40-Channel -->
-    <!--<VLP-16 parent="base_link"
-        name="velodyne"
-        topic="/velodyne_points"
-        hz="10"
-        samples="1000"
-        lasers="40"
-        collision_range ="0.3"
-        min_range ="0.3"
-        max_range ="200.0"
-        noise ="0.008"
-        min_angle="-${M_PI}"
-        max_angle="${M_PI}"
-        min_angle_ver="-16"
-        max_angle_ver="7"
-        >-->
-    <!-- simplified lidar for quick launch-->
-    <VLP-16 parent="base_link"
-            name="velodyne"
-            topic="/velodyne_points"
-            hz="8"
-            samples="1100"
-            lasers="36"
-            collision_range ="0.3"
-            min_range ="0.3"
-            max_range ="200.0"
-            noise ="0.1"
-            min_angle_hor="-${M_PI}"
-            max_angle_hor="${M_PI}"
-            min_angle_ver="-16"
-            max_angle_ver="7"
-            >
-      <origin xyz="0 0 0.4" rpy="0 0 0" />
-    </VLP-16>
-  </xacro:macro>
-  <xacro:velodyne_lidar />
   <gazebo>
     <plugin name="gazebo_ros_control" filename="libgazebo_ros_control.so">
